File: handBuilt Version/CabController_HB/SafetyLoop.kicad_sch (KiCad schematic)
At the start: 16 parts, among them J18 Screw_Terminal_01x02, J19 Conn_01x06, J28 SafetyLoop, U7 TLP293-4

Commit message: new TDU V2 page
Parts:
- removed J28: SafetyLoop, symbol Connector_Generic:Conn_02x05_Odd_Even
- added J29: Conn_01x09, symbol Connector_Generic:Conn_01x09
- added R28, R29: 1k, symbol Device:R
Connections:
- net GND: now also U7.11, U7.13, U7.15, U7.9, R28.2, R29.2
- net LV_sense: now also J29.9 (Pin_9); no longer U6.J3_13 (IN_1)
- net Sense1: now reaches U6.J3_8 (Sense1)
- net Sense1: now also J29.7 (Pin_7)
- net Sense2: now reaches U6.J3_18 (Sense2)
- net Sense2: now also J29.8 (Pin_8)
- net DI_4: now reaches R22.1, U7.16
- net DI_4: now also J29.4 (Pin_4)
- net HSO_2: now reaches U6.J3_14 (IN_2)
- net HSO_2: now also J29.6 (Pin_6)
- net DI_3: now reaches R23.1, U7.14
- net DI_3: now also J29.3 (Pin_3)
- net DI_1: now reaches R25.1, U7.10
- net DI_1: now also J29.1 (Pin_1)
- net DI_2: now reaches R24.1, U7.12
- net DI_2: now also J29.2 (Pin_2)
- net at J19.1 (Pin_1), U7.8: now also R28.1
- net at J19.2 (Pin_2), U7.6: now also R29.1
- new net HSO_1: J29.5 (Pin_5), U6.J3_13 (IN_1)
